File: NGL_Proto_ST_PCB/NGL_Proto_ST.sch (KiCad schematic (older format))
At the start: 52 parts, among them U1 AD8639, U2 AD8639, U3 MAX922CSAT

Commit message: Début ajout modifs de la review
Parts:
- R10P1: value 590 -> NC
- R2: value 442R -> 348R
- R2P1: value 1K -> NC
- TP1: value TestPoint -> IN
- TP2: value TestPoint -> IN_ADC
- TP3: value TestPoint -> OUT
- TP5: value TestPoint -> RECT
- TP6: renamed from TPP3; value TestPointPad -> CLK_GEN
Changed lines of the file:
@@
 P 2505 2000
 F 0 "R2" H 2575 2046 50  0000 L CNN
-F 1 "442R" H 2575 1955 50  0000 L CNN
+F 1 "348R" H 2575 1955 50  0000 L CNN
 F 2 "Resistor_SMD:R_0805_2012Metric_Pad1.20x1.40mm_HandSolder" V 2435 2000 50  0001 C CNN
 F 3 "~" H 2505 2000 50  0001 C CNN
@@
 P 9725 4785
 F 0 "TP2" H 9783 4903 50  0000 L CNN
-F 1 "TestPoint" H 9783 4812 50  0001 L CNN
+F 1 "IN_ADC" H 9783 4812 50  0000 L CNN
 F 2 "Connector_PinHeader_2.54mm:PinHeader_1x01_P2.54mm_Vertical" H 9925 4785 50  0001 C CNN
 F 3 "~" H 9925 4785 50  0001 C CNN
@@
 	1095 3215 1820 3215
 $Comp
-L Connector:TestPoint TPP3
+L Connector:TestPoint TP6
 U 1 1 62807395
 P 4420 2690
-F 0 "TPP3" H 4478 2808 50  0000 L CNN
-F 1 "TestPointPad" H 4478 2717 50  0001 L CNN
+F 0 "TP6" H 4478 2808 50  0000 L CNN
+F 1 "CLK_GEN" H 4460 2900 50  0000 L CNN
 F 2 "TestPoint:TestPoint_Pad_D3.0mm" H 4620 2690 50  0001 C CNN
 F 3 "~" H 4620 2690 50  0001 C CNN
@@
 P 7760 4785
 F 0 "TP5" H 7818 4903 50  0000 L CNN
-F 1 "TestPoint" H 7818 4812 50  0001 L CNN
+F 1 "RECT" H 7818 4812 50  0000 L CNN
 F 2 "Connector_PinHeader_2.54mm:PinHeader_1x01_P2.54mm_Vertical" H 7960 4785 50  0001 C CNN
 F 3 "~" H 7960 4785 50  0001 C CNN
@@
 P 3190 4720
 F 0 "TP3" H 3248 4838 50  0000 L CNN
-F 1 "TestPoint" H 3248 4747 50  0001 L CNN
+F 1 "OUT" H 3240 4740 50  0000 L CNN
 F 2 "Connector_PinHeader_2.54mm:PinHeader_1x01_P2.54mm_Vertical" H 3390 4720 50  0001 C CNN
 F 3 "~" H 3390 4720 50  0001 C CNN
@@
 U 1 1 62825857
 P 875 2655
-F 0 "TP1" H 933 2773 50  0000 L CNN
-F 1 "TestPoint" H 933 2682 50  0001 L CNN
+F 0 "TP1" V 960 2725 50  0000 L CNN
+F 1 "IN" V 780 2780 50  0000 L CNN
 F 2 "Connector_PinHeader_2.54mm:PinHeader_1x01_P2.54mm_Vertical" H 1075 2655 50  0001 C CNN
 F 3 "~" H 1075 2655 50  0001 C CNN
@@
 P 2500 1690
 F 0 "R2P1" H 2570 1736 50  0000 L CNN
-F 1 "1K" H 2570 1645 50  0000 L CNN
+F 1 "NC" H 2570 1645 50  0000 L CNN
 F 2 "Resistor_SMD:R_0805_2012Metric_Pad1.20x1.40mm_HandSolder" V 2430 1690 50  0001 C CNN
 F 3 "~" H 2500 1690 50  0001 C CNN
@@
 P 1775 4315
 F 0 "R10P1" H 1845 4361 50  0000 L CNN
-F 1 "590" H 1845 4270 50  0000 L CNN
+F 1 "NC" H 1845 4270 50  0000 L CNN
 F 2 "Resistor_SMD:R_0805_2012Metric_Pad1.20x1.40mm_HandSolder" V 1705 4315 50  0001 C CNN
 F 3 "~" H 1775 4315 50  0001 C CNN
