File: NGL_Proto_ST_PCB/Ampli Diff.sch (KiCad schematic (older format))
At the start: 30 parts, among them U7 AD620, U8 AD8639

Commit message: Début ajout modifs de la review
Parts:
- TP11: value TestPoint -> OUT_DIFF
- TP12: value TestPoint -> RECT_DIFF
- TP4: value TestPoint -> IN_ADC_DIFF
Changed lines of the file:
@@
 P 9310 3645
 F 0 "TP4" H 9368 3763 50  0000 L CNN
-F 1 "TestPoint" H 9368 3672 50  0001 L CNN
+F 1 "IN_ADC_DIFF" H 9368 3672 50  0000 L CNN
 F 2 "Connector_PinHeader_2.54mm:PinHeader_1x01_P2.54mm_Vertical" H 9510 3645 50  0001 C CNN
 F 3 "~" H 9510 3645 50  0001 C CNN
@@
 AR Path="/62B5BC1D/62828CD5" Ref="TP12"  Part="1"
 F 0 "TP12" H 7488 3763 50  0000 L CNN
-F 1 "TestPoint" H 7488 3672 50  0001 L CNN
+F 1 "RECT_DIFF" H 7488 3672 50  0000 L CNN
 F 2 "Connector_PinHeader_2.54mm:PinHeader_1x01_P2.54mm_Vertical" H 7630 3645 50  0001 C CNN
 F 3 "~" H 7630 3645 50  0001 C CNN
@@
 AR Path="/62B5BC1D/6282C25E" Ref="TP11"  Part="1"
 F 0 "TP11" H 2853 3908 50  0000 L CNN
-F 1 "TestPoint" H 2853 3817 50  0001 L CNN
+F 1 "OUT_DIFF" H 2630 4025 50  0000 L CNN
 F 2 "Connector_PinHeader_2.54mm:PinHeader_1x01_P2.54mm_Vertical" H 2995 3790 50  0001 C CNN
 F 3 "~" H 2995 3790 50  0001 C CNN
