File: NGL_Proto_ST_PCB/_autosave-Alim.sch (KiCad schematic (older format))
At the start: 21 parts, among them M1 ROB-08449, T1 RU1C002UNTCL, U5 LD29080PT33R, U6 MAX1680ESA+T

Commit message: GERBER généré: PRODUCTION
EURO
Parts:
- gave numbers to parts that had none: 1
Changed lines of the file:
@@
 P 1000 3615
 AR Path="/6271F3E2/62C95A99" Ref="R?"  Part="1"
-AR Path="/6271F3E2/62744FDF/62C95A99" Ref="R?"  Part="1"
-F 0 "R?" H 1070 3661 50  0000 L CNN
+AR Path="/6271F3E2/62744FDF/62C95A99" Ref="R18"  Part="1"
+F 0 "R18" H 1070 3661 50  0000 L CNN
 F 1 "4.7K" H 1070 3570 50  0000 L CNN
 F 2 "Resistor_SMD:R_0805_2012Metric_Pad1.20x1.40mm_HandSolder" V 930 3615 50  0001 C CNN
@@
 	1000 2810 1000 3465
 $Comp
-L power:GND #PWR?
+L power:GND #PWR067
 U 1 1 62C9B1A7
 P 1000 3990
-F 0 "#PWR?" H 1000 3740 50  0001 C CNN
+F 0 "#PWR067" H 1000 3740 50  0001 C CNN
 F 1 "GND" H 1005 3817 50  0000 C CNN
 F 2 "" H 1000 3990 50  0001 C CNN
